Commit message: add fc frame and root frame

File: gundam_rx78_description/urdf/GGC_TestModel_rx78_20170112.urdf (robot description, URDF)
Before this commit: robot GGC_TestModel_rx78_20170112, 98 links, 97 joints
Links:
- added link fc, mass 0.00001
- added link root, mass 0.00001
Joints:
- added joint fc_joint: type fixed, parent rx78_Null_018_link, child fc, origin xyz=0 0 0 rpy=0 0 0, axis 0 0 1
- added joint root_joint: type fixed, parent root, child base_link, origin xyz=0 0 0 rpy=0 0 0, axis 0 0 1
